Commit message: monster of a URDF file

File: urdf/rov.urdf (robot description, URDF)
Before this commit: robot rov, 24 links, 23 joints
Links:
- added link HGripper_Finger_Mobile, mass 0.034; collision box size=0.015 0.1 0.015; visual box size=0.015 0.1 0.015
- added link HGripper_Finger_Static, mass 0.034; collision box size=0.015 0.1 0.015; visual box size=0.015 0.1 0.015
- added link VGripper_Crossbar, mass 0.051000000000000004; collision box size=0.15 0.015 0.015; visual box size=0.15 0.015 0.015
- added link VGripper_Finger_Mobile, mass 0.034; collision box size=0.015 0.015 0.1; visual box size=0.015 0.015 0.1
- added link VGripper_Finger_Static, mass 0.034; collision box size=0.015 0.015 0.1; visual box size=0.015 0.015 0.1
- added link VGripper_Post, mass 0.034; collision box size=0.015 0.015 0.12; visual box size=0.015 0.015 0.12
- link Back_Left_Post: mass None -> 0.068; geometry collision box size=0.015 0.015 0.2; visual box size=0.015 0.015 0.2
- link Back_Right_Post: mass None -> 0.068; geometry collision box size=0.015 0.015 0.2; visual box size=0.015 0.015 0.2
- link HGripper_Crossbar: mass None -> 0.051000000000000004; geometry collision box size=0.15 0.015 0.015; visual box size=0.15 0.015 0.015
- link HGripper_Post: mass None -> 0.0408; geometry collision box size=0.015 0.12 0.015; visual box size=0.015 0.12 0.015
- link Left_Post: mass None -> 0.068; geometry collision box size=0.015 0.015 0.2; visual box size=0.015 0.015 0.2
- link Lower_Back_Crossbar: mass None -> 0.1258; geometry collision box size=0.37 0.015 0.015; visual box size=0.37 0.015 0.015
- link Lower_Front_Crossbar: mass None -> 0.1258; geometry collision box size=0.37 0.015 0.015; visual box size=0.37 0.015 0.015
- link Lower_Left_Crossbar: mass None -> 0.1394; geometry collision box size=0.015 0.41 0.015; visual box size=0.015 0.41 0.015
- link Lower_Right_Crossbar: mass None -> 0.1394; geometry collision box size=0.015 0.41 0.015; visual box size=0.015 0.41 0.015
- link MEH_Crossbar: mass None -> 0.1258; geometry collision box size=0.37 0.015 0.015; visual box size=0.37 0.015 0.015
- link PSE: mass None -> 1; geometry collision box size=0.17 0.12 0.055; visual box size=0.17 0.12 0.055
- link Right_Post: mass None -> 0.068; geometry collision box size=0.015 0.015 0.2; visual box size=0.015 0.015 0.2
- link SB_Left: mass None -> 0.3; geometry collision cylinder length=0.2 radius=0.055; visual cylinder length=0.2 radius=0.055
- link SB_Right: mass None -> 0.3; geometry collision cylinder length=0.2 radius=0.055; visual cylinder length=0.2 radius=0.055
- link Thruster_Back_Left: mass None -> 0.3; geometry collision cylinder length=0.05 radius=0.045; visual cylinder length=0.05 radius=0.045
- link Thruster_Back_Right: mass None -> 0.3; geometry collision cylinder length=0.05 radius=0.045; visual cylinder length=0.05 radius=0.045
- link Thruster_Front_Left: mass None -> 0.3; geometry collision cylinder length=0.05 radius=0.045; visual cylinder length=0.05 radius=0.045
- link Thruster_Front_Right: mass None -> 0.3; geometry collision cylinder length=0.05 radius=0.045; visual cylinder length=0.05 radius=0.045
- link Thruster_Vert_Left: mass None -> 0.3; geometry collision cylinder length=0.05 radius=0.045; visual cylinder length=0.05 radius=0.045
- link Thruster_Vert_Right: mass None -> 0.3; geometry collision cylinder length=0.05 radius=0.045; visual cylinder length=0.05 radius=0.045
- link Upper_Back_Crossbar: mass None -> 0.1258; geometry collision box size=0.37 0.015 0.015; visual box size=0.37 0.015 0.015
- link Upper_Left_Crossbar: mass None -> 0.1394; geometry collision box size=0.015 0.41 0.015; visual box size=0.015 0.41 0.015
- link Upper_Right_Crossbar: mass None -> 0.1394; geometry collision box size=0.015 0.41 0.015; visual box size=0.015 0.41 0.015
- link base_link: mass None -> 0.8; geometry collision box size=0.16 0.11 0.16; visual box size=0.16 0.11 0.16
Joints:
- added joint Bottom_Gripper: type prismatic, parent VGripper_Crossbar, child VGripper_Finger_Mobile, origin xyz=0.075 0 0, limit lower=-0.15 upper=0 effort=1000.0 velocity=0.5
- added joint Front_Gripper: type prismatic, parent HGripper_Crossbar, child HGripper_Finger_Mobile, origin xyz=0.075 0 0, limit lower=-0.15 upper=0 effort=1000.0 velocity=0.5
- added joint HGripper_Crossbar_HGF_Static: type fixed, parent HGripper_Crossbar, child HGripper_Finger_Static, origin xyz=-0.075 0 0
- added joint PSE_VGripper_Post: type fixed, parent PSE, child VGripper_Post, origin xyz=0 -0.12 0.03
- added joint VGripper_Crossbar_VGF_Static: type fixed, parent VGripper_Crossbar, child VGripper_Finger_Static, origin xyz=-0.075 0 0
- added joint VGripper_Post_VGripper_Crossbar: type fixed, parent VGripper_Post, child VGripper_Crossbar, origin xyz=0 0 -0.12
- joint HGripper_Post_HGripper_Crossbar: origin xyz=-0.1 -0.14 -0.125 -> xyz=0 -0.14 -0.125

File: urdf/rov.xacro (robot description, xacro)
@@ -3,4 +3,6 @@
 <!-- This is an .xacro file - that means it gets turned into a .urdf file
      after a couple of commands. It's used to simulate the ROV with ROS. -->
+  <!-- Some macros for making inertia definition easier-->
+  <xacro:include filename="inertial_macros.xacro"/>
   <!-- Xacro Properties Definition -->
   <!-- The following two properties are the
@@ -35,6 +37,16 @@
         <box size="0.16 0.11 0.16"/>
       </geometry>
-      <origin rpy="0 0 0" xyz="0 -0.055 0.04"/>
-    </visual>
+      <origin xyz="0 -0.055 0.04"/>
+      <material name="beige"/>
+    </visual>
+    <collision>
+      <geometry>
+        <box size="0.16 0.11 0.16"/>
+      </geometry>
+      <origin xyz="0 -0.055 0.04"/>
+    </collision>
+    <xacro:inertial_box mass="0.8" x="0.16" y="0.11" z="0.16">
+      <origin xyz="0 -0.055 0.04" rpy="0 0 0"/>
+    </xacro:inertial_box>
   </link>
   <!-- Upper Frame Definition -->
@@ -44,5 +56,14 @@
         <box size="${width} ${extrusion_width} ${extrusion_width}"/>
       </geometry>
-    </visual>
+      <material name="silver"/>
+    </visual>
+    <collision>
+      <geometry>
+        <box size="${width} ${extrusion_width} ${extrusion_width}"/>
+      </geometry>
+    </collision>
+    <xacro:inertial_box mass="${width * 0.34}" x="${width}" y="${extrusion_width}" z="${extrusion_width}">
+      <origin xyz="0 0 0" rpy="0 0 0"/>
+    </xacro:inertial_box>
   </link>
   <joint name="MEH_Crossbar_to_MEH" type="fixed">
@@ -55,6 +76,16 @@
         <box size="${extrusion_width} ${depth} ${extrusion_width}"/>
       </geometry>
-      <origin rpy="0 0 0" xyz="0 0.12 0"/>
-    </visual>
+      <material name="silver"/>
+      <origin rpy="0 0 0" xyz="0 0.12 0"/>
+    </visual>
+    <collision>
+      <geometry>
+        <box size="${extrusion_width} ${depth} ${extrusion_width}"/>
+      </geometry>
+      <origin rpy="0 0 0" xyz="0 0.12 0"/>
+    </collision>
+    <xacro:inertial_box mass="${depth * 0.34}" x="${extrusion_width}" y="${depth}" z="${extrusion_width}">
+      <origin xyz="0 0.12 0" rpy="0 0 0"/>
+    </xacro:inertial_box>
   </link>
   <joint name="MEH_Crossbar_UL_Crossbar" type="fixed">
@@ -68,6 +99,16 @@
         <box size="${extrusion_width} ${depth} ${extrusion_width}"/>
       </geometry>
-      <origin rpy="0 0 0" xyz="0 0.12 0"/>
-    </visual>
+      <material name="silver"/>
+      <origin rpy="0 0 0" xyz="0 0.12 0"/>
+    </visual>
+    <collision>
+      <geometry>
+        <box size="${extrusion_width} ${depth} ${extrusion_width}"/>
+      </geometry>
+      <origin rpy="0 0 0" xyz="0 0.12 0"/>
+    </collision>
+    <xacro:inertial_box mass="${depth * 0.34}" x="${extrusion_width}" y="${depth}" z="${extrusion_width}">
+      <origin xyz="0 0.12 0" rpy="0 0 0"/>
+    </xacro:inertial_box>
   </link>
   <joint name="MEH_Crossbar_UR_Crossbar" type="fixed">
@@ -81,6 +122,17 @@
         <box size="${width} ${extrusion_width} ${extrusion_width}"/>
       </geometry>
-      <origin xyz="${width / 2} 0 0"/>
-    </visual>
+      <material name="silver"/>
+      <origin xyz="${width / 2} 0 0"/>
+    </visual>
+    <collision>
+      <geometry>
+        <box size="${width} ${extrusion_width} ${extrusion_width}"/>
+      </geometry>
+      <material name="silver"/>
+      <origin xyz="${width / 2} 0 0"/>
+    </collision>
+    <xacro:inertial_box mass="${width*0.34}" x="${width}" y="${extrusion_width}" z="${extrusion_width}">
+      <origin xyz="${width / 2} 0 0"/>
+    </xacro:inertial_box>
   </link>
   <joint name="UB_Crossbar_UL_Crossbar" type="fixed">
@@ -90,11 +142,26 @@
   </joint>
   <!-- Vertical Frame Definition -->
+  <!-- Macros to quickly bang out the vertical posts-->
+  <xacro:macro name="frame_post">
+    <visual>
+      <geometry>
+        <box size="${extrusion_width} ${extrusion_width} ${height}"/>
+      </geometry>
+      <material name="silver"/>
+      <origin xyz="0 0 -${height / 2}"/>
+    </visual>
+    <collision>
+      <geometry>
+        <box size="${extrusion_width} ${extrusion_width} ${height}"/>
+      </geometry>
+      <material name="silver"/>
+      <origin xyz="0 0 -${height / 2}"/>
+    </collision>
+    <xacro:inertial_box mass="${height * 0.34}" x="${extrusion_width}" y="${extrusion_width}" z="${height}">
+      <origin xyz="0 0 -${height / 2}"/>
+    </xacro:inertial_box>
+  </xacro:macro>
   <link name="Left_Post">
-    <visual>
-      <geometry>
-        <box size="${extrusion_width} ${extrusion_width} ${height}"/>
-      </geometry>
-      <origin xyz="0 0 -${height / 2}"/>
-    </visual>
+    <xacro:frame_post/>
   </link>
   <joint name="UL_Crossbar_Left_Post" type="fixed">
@@ -103,10 +170,5 @@
   </joint>
   <link name="Right_Post">
-    <visual>
-      <geometry>
-        <box size="${extrusion_width} ${extrusion_width} ${height}"/>
-      </geometry>
-      <origin xyz="0 0 -${height / 2}"/>
-    </visual>
+    <xacro:frame_post/>
   </link>
   <joint name="UR_Crossbar_Right_Post" type="fixed">
@@ -115,10 +177,5 @@
   </joint>
   <link name="Back_Left_Post">
-    <visual>
-      <geometry>
-        <box size="${extrusion_width} ${extrusion_width} ${height}"/>
-      </geometry>
-      <origin xyz="0 0 -${height / 2}"/>
-    </visual>
+    <xacro:frame_post/>
   </link>
   <joint name="UL_Crossbar_BL_Post" type="fixed">
@@ -128,10 +185,5 @@
   </joint>
   <link name="Back_Right_Post">
-    <visual>
-      <geometry>
-        <box size="${extrusion_width} ${extrusion_width} ${height}"/>
-      </geometry>
-      <origin xyz="0 0 -${height / 2}"/>
-    </visual>
+    <xacro:frame_post/>
   </link>
   <joint name="UR_Crossbar_BR_Post" type="fixed">
@@ -146,6 +198,17 @@
         <box size="${width} ${extrusion_width} ${extrusion_width}"/>
       </geometry>
-      <origin xyz="${width / 2} 0 0"/>
-    </visual>
+      <material name="silver"/>
+      <origin xyz="${width / 2} 0 0"/>
+    </visual>
+    <collision>
+      <geometry>
+        <box size="${width} ${extrusion_width} ${extrusion_width}"/>
+      </geometry>
+      <material name="silver"/>
+      <origin xyz="${width / 2} 0 0"/>
+    </collision>
+    <xacro:inertial_box mass="${width * 0.34}" x="${width}" y="${extrusion_width}" z="${extrusion_width}">
+      <origin xyz="${width / 2} 0 0"/>
+    </xacro:inertial_box>
   </link>
   <joint name="LF_Crossbar_Left_Post" type="fixed">
@@ -159,6 +222,16 @@
         <box size="${extrusion_width} ${depth} ${extrusion_width}"/>
       </geometry>
-      <origin rpy="0 0 0" xyz="0 0.12 0"/>
-    </visual>
+      <material name="silver"/>
+      <origin rpy="0 0 0" xyz="0 0.12 0"/>
+    </visual>
+    <collision>
+      <geometry>
+        <box size="${extrusion_width} ${depth} ${extrusion_width}"/>
+      </geometry>
+      <origin rpy="0 0 0" xyz="0 0.12 0"/>
+    </collision>
+    <xacro:inertial_box mass="${depth*0.34}" x="${extrusion_width}" y="${depth}" z="${extrusion_width}">
+      <origin xyz="0 0.12 0" rpy="0 0 0"/>
+    </xacro:inertial_box>
   </link>
   <joint name="LF_Crossbar_LL_Crossbar" type="fixed">
@@ -172,6 +245,16 @@
         <box size="${extrusion_width} ${depth} ${extrusion_width}"/>
       </geometry>
-      <origin rpy="0 0 0" xyz="0 0.12 0"/>
-    </visual>
+      <material name="silver"/>
+      <origin rpy="0 0 0" xyz="0 0.12 0"/>
+    </visual>
+    <collision>
+      <geometry>
+        <box size="${extrusion_width} ${depth} ${extrusion_width}"/>
+      </geometry>
+      <origin rpy="0 0 0" xyz="0 0.12 0"/>
+    </collision>
+    <xacro:inertial_box mass="${depth*0.34}" x="${extrusion_width}" y="${depth}" z="${extrusion_width}">
+      <origin xyz="0 0.12 0" rpy="0 0 0"/>
+    </xacro:inertial_box>
   </link>
   <joint name="LF_Crossbar_LR_Crossbar" type="fixed">
@@ -185,6 +268,16 @@
         <box size="${width} ${extrusion_width} ${extrusion_width}"/>
       </geometry>
-      <origin xyz="${width / 2} 0 0"/>
-    </visual>
+      <material name="silver"/>
+      <origin xyz="${width / 2} 0 0"/>
+    </visual>
+    <collision>
+      <geometry>
+        <box size="${width} ${extrusion_width} ${extrusion_width}"/>
+      </geometry>
+      <origin xyz="${width / 2} 0 0"/>
+    </collision>
+    <xacro:inertial_box mass="${width*0.34}" x="${width}" y="${extrusion_width}" z="${extrusion_width}">
+      <origin xyz="${width / 2} 0 0"/>
+    </xacro:inertial_box>
   </link>
   <joint name="LB_Crossbar_LL_Crossbar" type="fixed">
@@ -199,6 +292,16 @@
         <box size="0.17 0.12 0.055"/>
       </geometry>
+      <material name="dark_gray"/>
       <origin xyz="0 -0.06 0.024"/>
     </visual>
+    <collision>
+      <geometry>
+        <box size="0.17 0.12 0.055"/>
+      </geometry>
+      <origin xyz="0 -0.06 0.024"/>
+    </collision>
+    <xacro:inertial_box mass="1" x="0.17" y="0.12" z="0.055">
+      <origin xyz="0 -0.06 0.024" rpy="0 0 0"/>
+    </xacro:inertial_box>
   </link>
   <joint name="UB_Crossbar_PSE" type="fixed">
@@ -212,6 +315,16 @@
         <cylinder length="0.2" radius="0.055"/>
       </geometry>
+      <material name="silver"/>
       <origin xyz="0 -0.045 -0.125"/>
     </visual>
+    <collision>
+      <geometry>
+        <cylinder length="0.2" radius="0.055"/>
+      </geometry>
+      <origin xyz="0 -0.045 -0.125"/>
+    </collision>
+    <xacro:inertial_cylinder mass="0.3" length="0.2" radius="0.055">
+      <origin rpy="0 0 0" xyz="0 -0.045 -0.125"/>
+    </xacro:inertial_cylinder>
   </link>
   <joint name="UB_Crossbar_SB_Left" type="fixed">
@@ -225,6 +338,17 @@
         <cylinder length="0.2" radius="0.055"/>
       </geometry>
+      <material name="silver"/>
       <origin xyz="0 -0.045 -0.125"/>
     </visual>
+    <collision>
+      <geometry>
+        <cylinder length="0.2" radius="0.055"/>
+      </geometry>
+      <material name="silver"/>
+      <origin xyz="0 -0.045 -0.125"/>
+    </collision>
+    <xacro:inertial_cylinder mass="0.3" length="0.2" radius="0.055">
+      <origin rpy="0 0 0" xyz="0 -0.045 -0.125"/>
+    </xacro:inertial_cylinder>
   </link>
   <joint name="UB_Crossbar_SB_Right" type="fixed">
@@ -234,11 +358,26 @@
   </joint>
   <!-- Thrusters -->
+  <!-- Macros to quickly bang out the identical thrusters-->
+  <xacro:macro name="horizontal_thruster">
+    <visual>
+      <geometry>
+        <cylinder length="0.05" radius="0.045"/>
+      </geometry>
+      <material name="black"/>
+      <origin rpy="1.57 0 0.77" xyz="0 0 -0.045"/>
+    </visual>
+    <collision>
+      <geometry>
+        <cylinder length="0.05" radius="0.045"/>
+      </geometry>
+      <material name="black"/>
+      <origin rpy="1.57 0 0.77" xyz="0 0 -0.045"/>
+    </collision>
+    <xacro:inertial_cylinder mass="0.3" length="0.05" radius="0.045">
+      <origin rpy="1.57 0 0.77" xyz="0 0 -0.045"/>
+    </xacro:inertial_cylinder>
+  </xacro:macro>
   <link name="Thruster_Front_Left">
-    <visual>
-      <geometry>
-        <cylinder length="0.05" radius="0.045"/>
-      </geometry>
-      <origin rpy="1.57 0 0.77" xyz="0 0 -0.045"/>
-    </visual>
+    <xacro:horizontal_thruster/>
   </link>
   <joint name="UL_Crossbar_TFL" type="fixed">
@@ -248,10 +387,5 @@
   </joint>
   <link name="Thruster_Back_Left">
-    <visual>
-      <geometry>
-        <cylinder length="0.05" radius="0.045"/>
-      </geometry>
-      <origin rpy="1.57 0 -0.77" xyz="0 0 -0.045"/>
-    </visual>
+    <xacro:horizontal_thruster/>
   </link>
   <joint name="UL_Crossbar_TBL" type="fixed">
@@ -261,10 +395,5 @@
   </joint>
   <link name="Thruster_Front_Right">
-    <visual>
-      <geometry>
-        <cylinder length="0.05" radius="0.045"/>
-      </geometry>
-      <origin rpy="1.57 0 -0.77" xyz="0 0 -0.045"/>
-    </visual>
+    <xacro:horizontal_thruster/>
   </link>
   <joint name="UR_Crossbar_TFR" type="fixed">
@@ -274,10 +403,5 @@
   </joint>
   <link name="Thruster_Back_Right">
-    <visual>
-      <geometry>
-        <cylinder length="0.05" radius="0.045"/>
-      </geometry>
-      <origin rpy="1.57 0 0.77" xyz="0 0 -0.045"/>
-    </visual>
+    <xacro:horizontal_thruster/>
   </link>
   <joint name="UR_Crossbar_TBR" type="fixed">
@@ -291,6 +415,16 @@
         <cylinder length="0.05" radius="0.045"/>
       </geometry>
+      <material name="black"/>
       <origin rpy="0 0 0" xyz="-0.045 0 0"/>
     </visual>
+    <collision>
+      <geometry>
+        <cylinder length="0.05" radius="0.045"/>
+      </geometry>
+      <origin rpy="0 0 0" xyz="-0.045 0 0"/>
+    </collision>
+    <xacro:inertial_cylinder mass="0.3" length="0.05" radius="0.045">
+      <origin rpy="0 0 0" xyz="-0.045 0 0"/>
+    </xacro:inertial_cylinder>
   </link>
   <joint name="UL_Crossbar_TVL" type="fixed">
@@ -304,6 +438,16 @@
         <cylinder length="0.05" radius="0.045"/>
       </geometry>
+      <material name="black"/>
       <origin rpy="0 0 0" xyz="0.045 0 0"/>
     </visual>
+    <collision>
+      <geometry>
+        <cylinder length="0.05" radius="0.045"/>
+      </geometry>
+      <origin rpy="0 0 0" xyz="0.045 0 0"/>
+    </collision>
+    <xacro:inertial_cylinder mass="0.3" length="0.05" radius="0.045">
+      <origin rpy="0 0 0" xyz="0.045 0 0"/>
+    </xacro:inertial_cylinder>
   </link>
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