Commit message: commit before URDF write

File: urdf/rov.gazebo.xacro (robot description, xacro)
@@ -1,13 +1,15 @@
-<?xml version="1.0" ?>
-<!-- =================================================================================== -->
-<!-- |    This document was autogenerated by xacro from rov.gazebo.xacro               | -->
-<!-- |    EDITING THIS FILE BY HAND IS NOT RECOMMENDED                                 | -->
-<!-- =================================================================================== -->
-<robot name="rov">
-  <!-- This is an .xacro file - that means it gets turned into a .urdf file
+<?xml version="1.0"?>
+<robot xmlns:xacro="http://www.ros.org/wiki/xacro" name="rov">
+<!-- This is an .xacro file - that means it gets turned into a .urdf file
      after a couple of commands. It's used to simulate the ROV with ROS. -->
-  <!-- Specify some standard inertial calculations https://en.wikipedia.org/wiki/List_of_moments_of_inertia -->
-  <!-- These make use of xacro's mathematical functionality -->
+  <!-- Some macros for making inertia definition easier-->
+  <xacro:include filename="inertial_macros.xacro"/>
   <!-- Xacro Properties Definition -->
+  <!-- The following two properties are the
+       dimensions of the 15x15mm frame-->
+  <xacro:property name="width" value = "0.37" />
+  <xacro:property name="depth" value = "0.41" />
+  <xacro:property name="height" value = "0.20" />
+  <xacro:property name="extrusion_width" value = "0.015" />
   <!-- Materials definition -->
   <material name="silver">
@@ -36,18 +38,16 @@
     <visual>
       <geometry>
-        <box size="0.37 0.015 0.015"/>
-      </geometry>
-      <material name="silver"/>
-    </visual>
-    <collision>
-      <geometry>
-        <box size="0.37 0.015 0.015"/>
-      </geometry>
-    </collision>
-    <inertial>
-      <origin rpy="0 0 0" xyz="0 0 0"/>
-      <mass value="0.1258"/>
-      <inertia ixx="4.717499999999999e-06" ixy="0.0" ixz="0.0" iyy="0.0014375270833333331" iyz="0.0" izz="0.0014375270833333331"/>
-    </inertial>
+        <box size="${width} ${extrusion_width} ${extrusion_width}"/>
+      </geometry>
+      <material name="silver"/>
+    </visual>
+    <collision>
+      <geometry>
+        <box size="${width} ${extrusion_width} ${extrusion_width}"/>
+      </geometry>
+    </collision>
+    <xacro:inertial_box mass="${width * 0.34}" x="${width}" y="${extrusion_width}" z="${extrusion_width}">
+      <origin xyz="0 0 0" rpy="0 0 0"/>
+    </xacro:inertial_box>
   </link>
   <joint name="Base_Link_MEH_Crossbar" type="fixed">
@@ -58,98 +58,94 @@
     <visual>
       <geometry>
-        <box size="0.015 0.41 0.015"/>
-      </geometry>
-      <material name="silver"/>
-      <origin rpy="0 0 0" xyz="0 0.12 0"/>
-    </visual>
-    <collision>
-      <geometry>
-        <box size="0.015 0.41 0.015"/>
-      </geometry>
-      <origin rpy="0 0 0" xyz="0 0.12 0"/>
-    </collision>
-    <inertial>
-      <origin rpy="0 0 0" xyz="0 0.12 0"/>
-      <mass value="0.1394"/>
-      <inertia ixx="0.001955375416666666" ixy="0.0" ixz="0.0" iyy="5.2274999999999995e-06" iyz="0.0" izz="0.001955375416666666"/>
-    </inertial>
+        <box size="${extrusion_width} ${depth} ${extrusion_width}"/>
+      </geometry>
+      <material name="silver"/>
+      <origin rpy="0 0 0" xyz="0 0.12 0"/>
+    </visual>
+    <collision>
+      <geometry>
+        <box size="${extrusion_width} ${depth} ${extrusion_width}"/>
+      </geometry>
+      <origin rpy="0 0 0" xyz="0 0.12 0"/>
+    </collision>
+    <xacro:inertial_box mass="${depth * 0.34}" x="${extrusion_width}" y="${depth}" z="${extrusion_width}">
+      <origin xyz="0 0.12 0" rpy="0 0 0"/>
+    </xacro:inertial_box>
   </link>
   <joint name="MEH_Crossbar_UL_Crossbar" type="fixed">
     <parent link="MEH_Crossbar"/>
     <child link="Upper_Left_Crossbar"/>
-    <origin xyz="-0.185 0 0"/>
+    <origin xyz="${-width / 2} 0 0"/>
   </joint>
   <link name="Upper_Right_Crossbar">
     <visual>
       <geometry>
-        <box size="0.015 0.41 0.015"/>
-      </geometry>
-      <material name="silver"/>
-      <origin rpy="0 0 0" xyz="0 0.12 0"/>
-    </visual>
-    <collision>
-      <geometry>
-        <box size="0.015 0.41 0.015"/>
-      </geometry>
-      <origin rpy="0 0 0" xyz="0 0.12 0"/>
-    </collision>
-    <inertial>
-      <origin rpy="0 0 0" xyz="0 0.12 0"/>
-      <mass value="0.1394"/>
-      <inertia ixx="0.001955375416666666" ixy="0.0" ixz="0.0" iyy="5.2274999999999995e-06" iyz="0.0" izz="0.001955375416666666"/>
-    </inertial>
+        <box size="${extrusion_width} ${depth} ${extrusion_width}"/>
+      </geometry>
+      <material name="silver"/>
+      <origin rpy="0 0 0" xyz="0 0.12 0"/>
+    </visual>
+    <collision>
+      <geometry>
+        <box size="${extrusion_width} ${depth} ${extrusion_width}"/>
+      </geometry>
+      <origin rpy="0 0 0" xyz="0 0.12 0"/>
+    </collision>
+    <xacro:inertial_box mass="${depth * 0.34}" x="${extrusion_width}" y="${depth}" z="${extrusion_width}">
+      <origin xyz="0 0.12 0" rpy="0 0 0"/>
+    </xacro:inertial_box>
   </link>
   <joint name="MEH_Crossbar_UR_Crossbar" type="fixed">
     <parent link="MEH_Crossbar"/>
     <child link="Upper_Right_Crossbar"/>
-    <origin xyz="0.185 0 0"/>
+    <origin xyz="${width / 2} 0 0"/>
   </joint>
   <link name="Upper_Back_Crossbar">
     <visual>
       <geometry>
-        <box size="0.37 0.015 0.015"/>
-      </geometry>
-      <material name="silver"/>
-      <origin xyz="0.185 0 0"/>
-    </visual>
-    <collision>
-      <geometry>
-        <box size="0.37 0.015 0.015"/>
-      </geometry>
-      <material name="silver"/>
-      <origin xyz="0.185 0 0"/>
-    </collision>
-    <inertial>
-      <origin xyz="0.185 0 0"/>
-      <mass value="0.1258"/>
-      <inertia ixx="4.717499999999999e-06" ixy="0.0" ixz="0.0" iyy="0.0014375270833333331" iyz="0.0" izz="0.0014375270833333331"/>
-    </inertial>
+        <box size="${width} ${extrusion_width} ${extrusion_width}"/>
+      </geometry>
+      <material name="silver"/>
+      <origin xyz="${width / 2} 0 0"/>
+    </visual>
+    <collision>
+      <geometry>
+        <box size="${width} ${extrusion_width} ${extrusion_width}"/>
+      </geometry>
+      <material name="silver"/>
+      <origin xyz="${width / 2} 0 0"/>
+    </collision>
+    <xacro:inertial_box mass="${width*0.34}" x="${width}" y="${extrusion_width}" z="${extrusion_width}">
+      <origin xyz="${width / 2} 0 0"/>
+    </xacro:inertial_box>
   </link>
   <joint name="UB_Crossbar_UL_Crossbar" type="fixed">
     <parent link="Upper_Left_Crossbar"/>
     <child link="Upper_Back_Crossbar"/>
-    <origin xyz="0 0.32999999999999996 0"/>
+    <origin xyz="0 ${depth - 0.08} 0"/>
   </joint>
   <!-- Vertical Frame Definition -->
+  <!-- Macros to quickly bang out the vertical posts-->
+  <xacro:macro name="frame_post">
+    <visual>
+      <geometry>
+        <box size="${extrusion_width} ${extrusion_width} ${height}"/>
+      </geometry>
+      <material name="silver"/>
+      <origin xyz="0 0 -${height / 2}"/>
+    </visual>
+    <collision>
+      <geometry>
+        <box size="${extrusion_width} ${extrusion_width} ${height}"/>
+      </geometry>
+      <material name="silver"/>
+      <origin xyz="0 0 -${height / 2}"/>
+    </collision>
+    <xacro:inertial_box mass="${height * 0.34}" x="${extrusion_width}" y="${extrusion_width}" z="${height}">
+      <origin xyz="0 0 -${height / 2}"/>
+    </xacro:inertial_box>
+  </xacro:macro>
   <link name="Left_Post">
-    <visual>
-      <geometry>
-        <box size="0.015 0.015 0.2"/>
-      </geometry>
-      <material name="silver"/>
-      <origin xyz="0 0 -0.1"/>
-    </visual>
-    <collision>
-      <geometry>
-        <box size="0.015 0.015 0.2"/>
-      </geometry>
-      <material name="silver"/>
-      <origin xyz="0 0 -0.1"/>
-    </collision>
-    <inertial>
-      <origin xyz="0 0 -0.1"/>
-      <mass value="0.068"/>
-      <inertia ixx="0.00022794166666666675" ixy="0.0" ixz="0.0" iyy="0.00022794166666666675" iyz="0.0" izz="2.55e-06"/>
-    </inertial>
+    <xacro:frame_post/>
   </link>
   <joint name="UL_Crossbar_Left_Post" type="fixed">
@@ -158,23 +154,5 @@
   </joint>
   <link name="Right_Post">
-    <visual>
-      <geometry>
-        <box size="0.015 0.015 0.2"/>
-      </geometry>
-      <material name="silver"/>
-      <origin xyz="0 0 -0.1"/>
-    </visual>
-    <collision>
-      <geometry>
-        <box size="0.015 0.015 0.2"/>
-      </geometry>
-      <material name="silver"/>
-      <origin xyz="0 0 -0.1"/>
-    </collision>
-    <inertial>
-      <origin xyz="0 0 -0.1"/>
-      <mass value="0.068"/>
-      <inertia ixx="0.00022794166666666675" ixy="0.0" ixz="0.0" iyy="0.00022794166666666675" iyz="0.0" izz="2.55e-06"/>
-    </inertial>
+    <xacro:frame_post/>
   </link>
   <joint name="UR_Crossbar_Right_Post" type="fixed">
@@ -183,54 +161,18 @@
   </joint>
   <link name="Back_Left_Post">
-    <visual>
-      <geometry>
-        <box size="0.015 0.015 0.2"/>
-      </geometry>
-      <material name="silver"/>
-      <origin xyz="0 0 -0.1"/>
-    </visual>
-    <collision>
-      <geometry>
-        <box size="0.015 0.015 0.2"/>
-      </geometry>
-      <material name="silver"/>
-      <origin xyz="0 0 -0.1"/>
-    </collision>
-    <inertial>
-      <origin xyz="0 0 -0.1"/>
-      <mass value="0.068"/>
-      <inertia ixx="0.00022794166666666675" ixy="0.0" ixz="0.0" iyy="0.00022794166666666675" iyz="0.0" izz="2.55e-06"/>
-    </inertial>
+    <xacro:frame_post/>
   </link>
   <joint name="UL_Crossbar_BL_Post" type="fixed">
     <parent link="Upper_Back_Crossbar"/>
     <child link="Back_Left_Post"/>
-    <origin xyz="0.111 0 0"/>
+    <origin xyz="${width * 0.3} 0 0"/>
   </joint>
   <link name="Back_Right_Post">
-    <visual>
-      <geometry>
-        <box size="0.015 0.015 0.2"/>
-      </geometry>
-      <material name="silver"/>
-      <origin xyz="0 0 -0.1"/>
-    </visual>
-    <collision>
-      <geometry>
-        <box size="0.015 0.015 0.2"/>
-      </geometry>
-      <material name="silver"/>
-      <origin xyz="0 0 -0.1"/>
-    </collision>
-    <inertial>
-      <origin xyz="0 0 -0.1"/>
-      <mass value="0.068"/>
-      <inertia ixx="0.00022794166666666675" ixy="0.0" ixz="0.0" iyy="0.00022794166666666675" iyz="0.0" izz="2.55e-06"/>
-    </inertial>
+    <xacro:frame_post/>
   </link>
   <joint name="UR_Crossbar_BR_Post" type="fixed">
     <parent link="Upper_Back_Crossbar"/>
     <child link="Back_Right_Post"/>
-    <origin xyz="0.259 0 0"/>
+    <origin xyz="${width * 0.7} 0 0"/>
   </joint>
   <!-- Lower Frame Definition -->
@@ -238,46 +180,42 @@
     <visual>
       <geometry>
-        <box size="0.37 0.015 0.015"/>
-      </geometry>
-      <material name="silver"/>
-      <origin xyz="0.185 0 0"/>
-    </visual>
-    <collision>
-      <geometry>
-        <box size="0.37 0.015 0.015"/>
-      </geometry>
-      <material name="silver"/>
-      <origin xyz="0.185 0 0"/>
-    </collision>
-    <inertial>
-      <origin xyz="0.185 0 0"/>
-      <mass value="0.1258"/>
-      <inertia ixx="4.717499999999999e-06" ixy="0.0" ixz="0.0" iyy="0.0014375270833333331" iyz="0.0" izz="0.0014375270833333331"/>
-    </inertial>
+        <box size="${width} ${extrusion_width} ${extrusion_width}"/>
+      </geometry>
+      <material name="silver"/>
+      <origin xyz="${width / 2} 0 0"/>
+    </visual>
+    <collision>
+      <geometry>
+        <box size="${width} ${extrusion_width} ${extrusion_width}"/>
+      </geometry>
+      <material name="silver"/>
+      <origin xyz="${width / 2} 0 0"/>
+    </collision>
+    <xacro:inertial_box mass="${width * 0.34}" x="${width}" y="${extrusion_width}" z="${extrusion_width}">
+      <origin xyz="${width / 2} 0 0"/>
+    </xacro:inertial_box>
   </link>
   <joint name="LF_Crossbar_Left_Post" type="fixed">
     <parent link="Left_Post"/>
     <child link="Lower_Front_Crossbar"/>
-    <origin xyz="0 0 -0.2"/>
+    <origin xyz="0 0 -${height}"/>
   </joint>
   <link name="Lower_Left_Crossbar">
     <visual>
       <geometry>
-        <box size="0.015 0.41 0.015"/>
-      </geometry>
-      <material name="silver"/>
-      <origin rpy="0 0 0" xyz="0 0.12 0"/>
-    </visual>
-    <collision>
-      <geometry>
-        <box size="0.015 0.41 0.015"/>
-      </geometry>
-      <origin rpy="0 0 0" xyz="0 0.12 0"/>
-    </collision>
-    <inertial>
-      <origin rpy="0 0 0" xyz="0 0.12 0"/>
-      <mass value="0.1394"/>
-      <inertia ixx="0.001955375416666666" ixy="0.0" ixz="0.0" iyy="5.2274999999999995e-06" iyz="0.0" izz="0.001955375416666666"/>
-    </inertial>
+        <box size="${extrusion_width} ${depth} ${extrusion_width}"/>
+      </geometry>
+      <material name="silver"/>
+      <origin rpy="0 0 0" xyz="0 0.12 0"/>
+    </visual>
+    <collision>
+      <geometry>
+        <box size="${extrusion_width} ${depth} ${extrusion_width}"/>
+      </geometry>
+      <origin rpy="0 0 0" xyz="0 0.12 0"/>
+    </collision>
+    <xacro:inertial_box mass="${depth*0.34}" x="${extrusion_width}" y="${depth}" z="${extrusion_width}">
+      <origin xyz="0 0.12 0" rpy="0 0 0"/>
+    </xacro:inertial_box>
   </link>
   <joint name="LF_Crossbar_LL_Crossbar" type="fixed">
@@ -289,50 +227,46 @@
     <visual>
       <geometry>
-        <box size="0.015 0.41 0.015"/>
-      </geometry>
-      <material name="silver"/>
-      <origin rpy="0 0 0" xyz="0 0.12 0"/>
-    </visual>
-    <collision>
-      <geometry>
-        <box size="0.015 0.41 0.015"/>
-      </geometry>
-      <origin rpy="0 0 0" xyz="0 0.12 0"/>
-    </collision>
-    <inertial>
-      <origin rpy="0 0 0" xyz="0 0.12 0"/>
-      <mass value="0.1394"/>
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